Commit message: Added revolute gripper joint

File: UR3e_RG2_ER5_description/urdf/rg2.urdf.xacro (robot description, xacro)
@@ -31,9 +31,17 @@
       </inertial>
     </link>
-    <joint name="rg2_eef_joint" type="fixed">
+    <!--joint name="rg2_eef_joint" type="fixed">
       <origin rpy="0 0 0" xyz="0.195 0.0 0.0"/>
       <parent link="rg2_body_link"/>
       <child link="rg2_eef_link"/>
     </joint>
+    <link name="rg2_eef_link"/-->
+    <joint name="gripper_joint" type="revolute">
+      <origin rpy="0 0 0" xyz="0.195 0.0 0.0"/>
+      <parent link="rg2_body_link"/>
+      <child link="rg2_eef_link"/>
+      <axis  xyz="1 0 0" />
+      <limit effort="1" lower="-1" upper="1" velocity="1"/>
+    </joint>
     <link name="rg2_eef_link"/>
   </xacro:macro>

Commit message: Added gripper_joint transmission to fix controller

File: UR3e_RG2_ER5_description/urdf/rg2.urdf.xacro (robot description, xacro)
@@ -3,11 +3,10 @@
 <robot name="rg2" xmlns:xacro="http://ros.org/wiki/xacro">
   <xacro:macro name="rg2" params="prefix">
-    <link name="gripper_extender_link" />
-    <!-- rg2 joint -->
+    <!--link name="gripper_extender_link" />
     <joint name="rg2_joint" type="fixed">
       <origin rpy="0 -1.57 0" xyz="0 0 0"/>
       <parent link="${prefix}gripper_extender_link"/>
       <child link="${prefix}rg2_body_link"/>
-    </joint>
+    </joint-->
     <link name="${prefix}rg2_body_link">
       <visual>
@@ -39,10 +38,19 @@
     <joint name="gripper_joint" type="revolute">
       <origin rpy="0 0 0" xyz="0.195 0.0 0.0"/>
+      <axis  xyz="0 0 1" />
+      <limit effort="1000" lower="0" upper=".548" velocity="0.5"/>
       <parent link="rg2_body_link"/>
       <child link="rg2_eef_link"/>
-      <axis  xyz="1 0 0" />
-      <limit effort="1" lower="-1" upper="1" velocity="1"/>
     </joint>
     <link name="rg2_eef_link"/>
+    <transmission name="gripper_joint_trans">
+      <type>transmission_interface/SimpleTransmission</type>
+      <joint name="gripper_joint">
+        <hardwareInterface>hardware_interface/PositionJointInterface</hardwareInterface>
+      </joint>
+      <actuator name="gripper_joint_motor">
+        <mechanicalReduction>1</mechanicalReduction>
+      </actuator>
+    </transmission>
   </xacro:macro>
 </robot>

File: UR3e_RG2_ER5_description/urdf/ur3e_with_rg2.urdf.xacro (robot description, xacro)
@@ -24,8 +24,9 @@
   </joint>
   <joint name="ur3e_to_gripper" type="fixed">
-    <origin xyz="0 0 0.0" rpy="0 0 0"/>
+    <origin xyz="0 0 0.0" rpy="0 ${-pi/2} 0"/>
     <parent link="tool0"/>
     <parent link="wrist_3_link" />
-    <child link="gripper_extender_link"/>
+    <!--child link="gripper_extender_link"/-->
+    <child link="rg2_body_link"/>
   </joint>
   <link name="world" />

Commit message: Fixed gripper controller issues

File: UR3e_RG2_ER5_description/urdf/rg2.urdf.xacro (robot description, xacro)
@@ -43,5 +43,10 @@
       <child link="rg2_eef_link"/>
     </joint>
-    <link name="rg2_eef_link"/>
+    <link name="rg2_eef_link">
+    <inertial>
+        <mass value="1"/>
+        <inertia ixx="1" ixy="0.0" ixz="0.0" iyy="1" iyz="0.0" izz="1"/>
+      </inertial>
+    </link>
     <transmission name="gripper_joint_trans">
       <type>transmission_interface/SimpleTransmission</type>
