Commit message: Fixed collision objects

File: UR3e_RG2_ER5_description/urdf/er5.urdf.xacro (robot description, xacro)
@@ -15,4 +15,11 @@
       <collision>
 <!--        <origin rpy="1.57 0 3.14" xyz="0.53 -0.27 -1.05"/> -->
+        <origin rpy="0 0 0" xyz="-0.12 0.0 -.3"/>
+        <geometry>
+          <cylinder length="0.6" radius="0.2"/>
+        </geometry>
+      </collision>
+      <collision>
+<!--        <origin rpy="1.57 0 3.14" xyz="0.53 -0.27 -1.05"/> -->
         <origin rpy="0 0 0" xyz=".30 0 -.625"/>
         <geometry>

File: UR3e_RG2_ER5_description/urdf/rg2.urdf.xacro (robot description, xacro)
@@ -21,7 +21,7 @@
       </visual>
       <collision>
-        <origin rpy="0 1.57 0" xyz="0.1 0.0085 0.0"/>
+        <origin rpy="0 1.57 0" xyz="0.1 0.0 0.0"/>
         <geometry>
-          <cylinder length="0.05" radius="0.03"/>
+          <cylinder length="0.2" radius="0.05"/>
         </geometry>
       </collision>

Commit message: Added gripper_joint to pick-and-place

File: UR3e_RG2_ER5_description/urdf/er5.urdf.xacro (robot description, xacro)
@@ -17,5 +17,5 @@
         <origin rpy="0 0 0" xyz="-0.12 0.0 -.3"/>
         <geometry>
-          <cylinder length="0.6" radius="0.2"/>
+          <cylinder length="0.6" radius="0.1"/>
         </geometry>
       </collision>

Commit message: Added descriptions and instructions.

File: UR3e_RG2_ER5_description/urdf/er5.urdf.xacro (robot description, xacro)
@@ -13,11 +13,10 @@
         </material>
       </visual>
-      <collision>
-<!--        <origin rpy="1.57 0 3.14" xyz="0.53 -0.27 -1.05"/> -->
+      <!--collision>
         <origin rpy="0 0 0" xyz="-0.12 0.0 -.3"/>
         <geometry>
-          <cylinder length="0.6" radius="0.1"/>
+          <cylinder length="0.6" radius="0.2"/>
         </geometry>
-      </collision>
+      </collision-->
       <collision>
 <!--        <origin rpy="1.57 0 3.14" xyz="0.53 -0.27 -1.05"/> -->

File: UR3e_RG2_ER5_description/urdf/rg2.urdf.xacro (robot description, xacro)
@@ -39,5 +39,5 @@
       <origin rpy="0 0 0" xyz="0.195 0.0 0.0"/>
       <axis  xyz="0 0 1" />
-      <limit effort="1000" lower="0" upper=".548" velocity="0.5"/>
+      <limit effort="1000" lower="0" upper="3.14" velocity="3.14"/>
       <parent link="rg2_body_link"/>
       <child link="rg2_eef_link"/>

Commit message: staging for Github

File: UR3e_RG2_ER5_description/urdf/er5.urdf.xacro (robot description, xacro)
@@ -13,10 +13,10 @@
         </material>
       </visual>
-      <!--collision>
+      <collision>
         <origin rpy="0 0 0" xyz="-0.12 0.0 -.3"/>
         <geometry>
           <cylinder length="0.6" radius="0.2"/>
         </geometry>
-      </collision-->
+      </collision>
       <collision>
 <!--        <origin rpy="1.57 0 3.14" xyz="0.53 -0.27 -1.05"/> -->

File: UR3e_RG2_ER5_description/urdf/rg2.urdf.xacro (robot description, xacro)
@@ -22,5 +22,5 @@
         <origin rpy="0 1.57 0" xyz="0.1 0.0 0.0"/>
         <geometry>
-          <cylinder length="0.2" radius="0.05"/>
+          <cylinder length="0.1" radius="0.05"/>
         </geometry>
       </collision>

File: UR3e_RG2_ER5_pick_place/urdf/object_sphere.urdf.xacro (robot description, xacro)
@@ -1,4 +1,4 @@
-<robot name="object">
-  <link name="object">
+<robot name="sphere">
+  <link name="sphere">
     <inertial>
       <origin xyz="0.35 0 0" />
@@ -9,5 +9,5 @@
       <origin xyz="0.35 0 0.65"/>
       <geometry>
-        <box size="0.02 0.02 0.2" />
+        <sphere radius=1 />
       </geometry>
     </visual>
@@ -15,9 +15,9 @@
       <origin xyz="0.35 0 0.65"/>
       <geometry>
-        <box size="0.02 0.02 0.2" />
+        <sphere radius=1 />
       </geometry>
     </collision>
   </link>
-  <gazebo reference="object">
+  <gazebo reference="sphere">
     <material>Gazebo/Green</material>
   </gazebo>
